Commit message: feat(urdf, meshes): updates urdf, meshes model and README (gmy)

File: urdf/left.urdf (robot description, URDF)
Before this commit: robot wujihand-left-v1.0.0, 26 links, 25 joints
Joints:
- joint finger1_joint1: axis -0 1 -0 -> 0 0 -1; limit lower=-0.0448 upper=1.6508 effort=0.6 velocity=8.58701992 -> lower=-1.6508 upper=0.0448 effort=0.6 velocity=8.587; origin xyz=0.0085244 -0.020575 0.028712 rpy=1.328 -0.37161 0.7307 -> xyz=0.0085244 -0.020575 0.028712 rpy=0.38179 -0.2259 -0.92978
- joint finger1_joint2: axis -1 0 0 -> 0 0 -1; limit lower=-0.1659 upper=0.9339 effort=0.6 velocity=11.10029404 -> lower=-0.1659 upper=0.9339 effort=0.6 velocity=11.1; origin xyz=-0.0047549 0.0060191 0.014132 rpy=-0.27968 -0.55633 -0.081982 -> xyz=0.014132 -0.0047549 0.0060191 rpy=-1.6442 -0.32223 -0.53456
- joint finger1_joint3: axis 0 1 0 -> 0 0 1; limit lower=-0.4932 upper=1.6272 effort=0.3 velocity=12.86307659 -> lower=-0.4932 upper=1.6272 effort=0.3 velocity=12.863; origin xyz=0.0009915 -0.00026671 0.033166 rpy=-0.049049 0.017311 0.33774 -> xyz=0.034664 0.00018873 0.0009916 rpy=1.909 -6.6317E-05 -0.052012
- joint finger1_joint4: axis 0 1 0 -> 0 0 1; limit lower=-0.4932 upper=1.6272 effort=0.3 velocity=13.57866158 -> lower=-0.4932 upper=1.6272 effort=0.3 velocity=13.579; origin xyz=0 4.0225E-05 0.028987 rpy=0 0 0 -> xyz=0.0295 0 0.00025125 rpy=0 0 0
- joint finger1_tip_fixed: limit lower=-0.5236 upper=0.5236 effort=100 velocity=10 -> (none); origin xyz=-0.001058 -0.00044022 0.029313 rpy=0 0 0 -> xyz=0.0283 -0.0010446 -0.00024656 rpy=0 0 0
- joint finger2_joint1: axis 0 1 0 -> 1 0 0; limit lower=-0.32695 upper=1.63595 effort=1 velocity=8.203047484 -> lower=-0.32695 upper=1.636 effort=1 velocity=8.203; origin xyz=-0.0058701 -0.029434 0.091917 rpy=0.11071 -0.071133 0.21823 -> xyz=-0.0058701 -0.029434 0.091917 rpy=-0.071558 -0.11043 1.7969
- joint finger2_joint2: axis -1 -0 -0 -> 0 0 1; limit lower=-0.495 upper=0.495 effort=0.2 velocity=8.115781022 -> lower=-0.495 upper=0.495 effort=0.2 velocity=8.1158; origin xyz=0.0022 0 0.004 rpy=-0.00043322 1.0969E-05 0 -> xyz=0 -0.0022 0.004 rpy=1.5708 -1.5708 0
- joint finger2_joint3: axis -0 1 -0 -> 0 0 -1; limit lower=-0.4932 upper=1.6272 effort=0.3 velocity=12.86307659 -> lower=-1.6272 upper=0.4932 effort=0.3 velocity=12.863; origin xyz=-0.0046 0 0.036618 rpy=0 0 -0.00026861 -> xyz=0.043618 0 -0.00475 rpy=1.5705 0 0
- joint finger2_joint4: axis -0 1 -0 -> 0 0 -1; limit lower=-0.4932 upper=1.6272 effort=0.3 velocity=13.57866158 -> lower=-1.6272 upper=0.4932 effort=0.3 velocity=13.579; origin xyz=0 0 0.029 rpy=0 0 0 -> xyz=0.0295 0 0 rpy=0 0 0
- joint finger2_tip_fixed: origin xyz=-0.0010404 0 0.0267 rpy=0 0 0 -> xyz=0.0267 -0.00105 0 rpy=0 0 0
- joint finger3_joint1: axis -0 1 -0 -> -1 0 0; limit lower=-0.32695 upper=1.63595 effort=1 velocity=8.203047484 -> lower=-1.63595 upper=0.32695 effort=1 velocity=8.203; origin xyz=-0.01046 -0.0074615 0.089544 rpy=5.0886E-05 -0.087266 -0.00058387 -> xyz=-0.01046 -0.0074615 0.089544 rpy=-0.087266 -5.0693E-05 1.5702
- joint finger3_joint2: axis -1 0 0 -> 0 0 -1; limit lower=-0.495 upper=0.495 effort=0.2 velocity=8.115781022 -> lower=-0.495 upper=0.495 effort=0.2 velocity=8.115; origin xyz=0.0022 0 0.004 rpy=-0.00043323 0 0 -> xyz=0 -0.0022 0.004 rpy=1.5708 -1.5708 0
- joint finger3_joint3: axis -0 1 -0 -> 0 0 -1; limit lower=-0.4932 upper=1.6272 effort=0.3 velocity=12.86307659 -> lower=-1.6272 upper=0.4932 effort=0.3 velocity=12.863; origin xyz=-0.0046 0 0.036618 rpy=0 0 -0.00026862 -> xyz=0.043618 0 -0.00475 rpy=1.5705 0 0
- joint finger3_joint4: axis -0 1 -0 -> 0 0 -1; limit lower=-0.4932 upper=1.6272 effort=0.3 velocity=13.57866158 -> lower=-1.6272 upper=0.4932 effort=0.3 velocity=13.579; origin xyz=0 0 0.029 rpy=0 0 0 -> xyz=0.0295 0 0 rpy=0 0 0
- joint finger3_tip_fixed: origin xyz=-0.0010404 0 0.0267 rpy=0 0 0 -> xyz=0.0267 -0.0010501 0 rpy=0 0 0
- joint finger4_joint1: axis -0 1 -0 -> -1 0 0; limit lower=-0.32695 upper=1.63595 effort=1 velocity=8.203047484 -> lower=-1.63595 upper=0.32695 effort=1 velocity=8.203; origin xyz=-0.0076649 0.013712 0.084429 rpy=-0.090379 -0.084038 -0.047072 -> xyz=-0.0076649 0.013712 0.084429 rpy=-0.083776 0.090059 1.5161
- joint finger4_joint2: axis -1 0 0 -> 0 0 -1; limit lower=-0.495 upper=0.495 effort=0.2 velocity=8.115781022 -> lower=-0.495 upper=0.495 effort=0.2 velocity=8.1158; origin xyz=0.0022024 0 0.0039987 rpy=-0.00043323 0.00060486 0 -> xyz=0 -0.0022 0.004 rpy=1.5708 -1.5708 0
- joint finger4_joint3: axis -0 1 -0 -> 0 0 -1; limit lower=-0.4932 upper=1.6272 effort=0.3 velocity=12.86307659 -> lower=-1.6272 upper=0.4932 effort=0.3 velocity=12.863; origin xyz=-0.0046 0 0.036618 rpy=0 0 -0.00026862 -> xyz=0.043618 0 -0.00475 rpy=1.5705 0 0
- joint finger4_joint4: axis -0 1 -0 -> 0 0 -1; limit lower=-0.4932 upper=1.6272 effort=0.3 velocity=13.57866158 -> lower=-1.6272 upper=0.4932 effort=0.3 velocity=13.579; origin xyz=0 0 0.029 rpy=0 0 0 -> xyz=0.0295 0 0 rpy=0 0 0
- joint finger4_tip_fixed: origin xyz=-0.0010993 0 0.026698 rpy=0 0 0 -> xyz=0.0267 -0.0010573 0 rpy=0 0 0
- joint finger5_joint1: axis 0 1 0 -> 1 0 0; limit lower=-0.32695 upper=1.63595 effort=1 velocity=8.203047484 -> lower=-0.32695 upper=1.636 effort=1 velocity=8.203; origin xyz=-0.0022687 0.034001 0.074281 rpy=-0.1925 -0.09326 -0.15753 -> xyz=-0.0022687 0.034001 0.074281 rpy=-0.094248 0.19165 1.3951
- joint finger5_joint2: axis -1 0 0 -> 0 0 -1; limit lower=-0.495 upper=0.495 effort=0.2 velocity=8.115781022 -> lower=-0.495 upper=0.495 effort=0.2 velocity=8.1158; origin xyz=0.002203 0 0.0039983 rpy=-0.00043323 0.00075655 0 -> xyz=0 -0.0022 0.004 rpy=-0.0067566 -1.5708 1.5776
- joint finger5_joint3: axis -0 1 -0 -> 0 0 -1; limit lower=-0.4932 upper=1.6272 effort=0.3 velocity=12.86307659 -> lower=-1.6272 upper=0.4932 effort=0.3 velocity=12.863; origin xyz=-0.0046 0 0.036618 rpy=0 0 -0.00026862 -> xyz=0.043618 0 -0.00475 rpy=1.5705 0 0
- joint finger5_joint4: axis -0 1 -0 -> 0 0 1; limit lower=-0.4932 upper=1.6272 effort=0.3 velocity=13.57866158 -> lower=-0.4932 upper=1.6272 effort=0.3 velocity=13.579; origin xyz=0 0 0.029 rpy=0 0 0 -> xyz=0.0295 0 0 rpy=0 0 0
- joint finger5_tip_fixed: limit effort=100 velocity=10 -> (none); origin xyz=-0.0011127 0 0.026697 rpy=0 0 0 -> xyz=0.0267 -0.0010582 0 rpy=0 0 0

File: urdf/right.urdf (robot description, URDF)
Before this commit: robot wujihand-right-v1.0.0, 26 links, 25 joints
Joints:
- joint finger1_joint1: axis -0 1 -0 -> 0 -1 0; limit lower=-0.0448 upper=1.6508 effort=0.6 velocity=8.58701992 -> lower=-1.6508 upper=0.0448 effort=0.6 velocity=8.587; origin xyz=0.00852444051536966 0.0205754004992104 0.0287119465316217 rpy=-1.32802443797267 -0.371613529401197 -0.730700470955738 -> xyz=0.0085244 0.020575 0.028712 rpy=-1.328 -0.37161 -0.7307
- joint finger1_joint2: axis -0 -1 -0 -> 0 1 0; limit lower=-0.1659 upper=0.9339 effort=0.6 velocity=11.10029404 -> lower=-0.9339 upper=0.1659 effort=0.6 velocity=11.1; origin xyz=-0.00475489770145063 -0.00601914141399163 0.0141320977109324 rpy=-0.574275025049342 -0.236773483165492 1.80339766411149 -> xyz=-0.0047549 -0.0060191 0.014132 rpy=-0.57428 -0.23677 1.8034
- joint finger1_joint3: limit lower=-0.4932 upper=1.6272 effort=0.3 velocity=12.86307659 -> lower=-0.4932 upper=1.6272 effort=0.3 velocity=12.863; origin xyz=0.00026670985188593 -0.000991501581071832 0.0331656190850421 rpy=0.0490494507279603 0.0173112436656061 -1.90854042682209 -> xyz=0.00018873 -0.0009916 0.034664 rpy=0.049049 0.017311 -1.9085
- joint finger1_joint4: limit lower=-0.4932 upper=1.6272 effort=0.3 velocity=13.57866158 -> lower=-0.4932 upper=1.6272 effort=0.3 velocity=13.579; origin xyz=0 -5.00007422951686E-05 0.0289999996622586 rpy=0 0 0 -> xyz=0 -0.00025 0.0295 rpy=0 0 0
- joint finger1_tip_fixed: limit lower=0 upper=0 effort=100 velocity=10 -> (none); origin xyz=-0.00104623528319934 0.000443681117589321 0.0293000000558906 rpy=0 0 0 -> xyz=-0.0011048 0.00023218 0.0283 rpy=0 0 0
- joint finger2_joint1: axis 0 0.999999906158207 0.000433224625971368 -> 0 1 0; limit lower=-0.32695 upper=1.63595 effort=1 velocity=8.203047484 -> lower=-0.32695 upper=1.636 effort=1 velocity=8.203; origin xyz=-0.00587008921485247 0.0294338632809287 0.0919165306699325 rpy=-0.111142508461784 -0.0711392477320386 -0.218224846477167 -> xyz=-0.0058701 0.029434 0.091917 rpy=-0.11071 -0.071139 -0.21822
- joint finger2_joint2: axis -0.999999999978991 0 0 -> -1 0 0; limit lower=-0.495 upper=0.495 effort=0.2 velocity=8.115781022 -> lower=-0.495 upper=0.495 effort=0.2 velocity=8.1158; origin xyz=0.00220000017524629 0 0.00400000534382478 rpy=0.000433224548403847 0 0 -> xyz=0.0022 0 0.004 rpy=0 0 0
- joint finger2_joint3: axis -0 1 -0 -> 0 -1 0; limit lower=-0.4932 upper=1.6272 effort=0.3 velocity=12.86307659 -> lower=-1.6272 upper=0.4932 effort=0.3 velocity=12.863; origin xyz=-0.00460023735005808 1.55817705260984E-05 0.0366176526568538 rpy=-0.000433222790942502 0 -0.000268612691124751 -> xyz=-0.0047503 0 0.043618 rpy=0 0 -0.00026861
- joint finger2_joint4: axis -0 1 -0 -> 0 -1 0; limit lower=-0.4932 upper=1.6272 effort=0.3 velocity=13.57866158 -> lower=-1.6272 upper=0.4932 effort=0.3 velocity=13.579; origin xyz=0 0 0.0290000000150095 rpy=0 0 0 -> xyz=0 0 0.0295 rpy=0 0 0
- joint finger2_tip_fixed: limit lower=0 upper=0 effort=100 velocity=10 -> (none); origin xyz=-0.00104999539509563 0 0.0274000004481596 rpy=0 0 0 -> xyz=-0.00105 0 0.0274 rpy=0 0 0
- joint finger3_joint1: axis 0 0.999999906158095 0.000433224884501103 -> 0 1 0; limit lower=-0.32695 upper=1.63595 effort=1 velocity=8.203047484 -> lower=-0.32695 upper=1.636 effort=1 velocity=8.203; origin xyz=-0.0104597238611628 0.00746146014385576 0.0895435117703666 rpy=-0.00048411119168703 -0.087266465303481 0.000583871740106801 -> xyz=-0.01046 0.0074615 0.089544 rpy=-5.0886E-05 -0.087266 0.00058387
- joint finger3_joint2: limit lower=-0.495 upper=0.495 effort=0.2 velocity=8.115781022 -> lower=-0.495 upper=0.495 effort=0.2 velocity=8.1158; origin xyz=0.0022000005026625 0 0.00400000522628907 rpy=0.000433224806924388 0 0 -> xyz=0.0022 0 0.004 rpy=0 0 0
- joint finger3_joint3: axis -0 1 -0 -> 0 -1 0; limit lower=-0.4932 upper=1.6272 effort=0.3 velocity=12.86307659 -> lower=-1.6272 upper=0.4932 effort=0.3 velocity=12.863; origin xyz=-0.00460000064410125 1.55817799863825E-05 0.036617682393194 rpy=-0.000433224785853114 0 -0.000268612686864552 -> xyz=-0.00475 0 0.043618 rpy=0 0 -0.00026861
- joint finger3_joint4: axis -0 1 -0 -> 0 -1 0; limit lower=-0.4932 upper=1.6272 effort=0.3 velocity=13.57866158 -> lower=-1.6272 upper=0.4932 effort=0.3 velocity=13.579; origin xyz=0 0 0.0290000000150094 rpy=0 0 0 -> xyz=0 0 0.0295 rpy=0 0 0
- joint finger3_tip_fixed: limit lower=0 upper=0 effort=100 velocity=10 -> (none); origin xyz=-0.00104042865141054 0 0.0267000008801756 rpy=0 0 0 -> xyz=-0.0010491 0 0.0267 rpy=0 0 0
- joint finger4_joint1: axis 0 0.999999906157892 0.000433225355001288 -> 0 -1 0; limit lower=-0.32695 upper=1.63595 effort=1 velocity=8.203047484 -> lower=-1.63595 upper=0.32695 effort=1 velocity=8.203; origin xyz=-0.0076648599285041 -0.0137122383759844 0.084428694586379 rpy=0.0899413960034348 -0.0834355049367681 0.0471266288536016 -> xyz=-0.0076649 -0.013712 0.084429 rpy=0.090375 -0.083436 0.047127
- joint finger4_joint2: limit lower=-0.495 upper=0.495 effort=0.2 velocity=8.115781022 -> lower=-0.495 upper=0.495 effort=0.2 velocity=8.1158; origin xyz=0.00220000053755089 0 0.00400000510026774 rpy=0.000433225366118357 0 0 -> xyz=0.0022 0 0.004 rpy=0 0 0
- joint finger4_joint3: axis -0 1 -0 -> 0 -1 0; limit lower=-0.4932 upper=1.6272 effort=0.3 velocity=12.86307659 -> lower=-1.6272 upper=0.4932 effort=0.3 velocity=12.863; origin xyz=-0.00459999999033558 1.55818004638833E-05 0.0366176824753135 rpy=-0.000433225349833524 0 -0.000268612687102299 -> xyz=-0.00475 0 0.043618 rpy=0 0 -0.00026861
- joint finger4_joint4: axis -0 1 -0 -> 0 -1 0; limit lower=-0.4932 upper=1.6272 effort=0.3 velocity=13.57866158 -> lower=-1.6272 upper=0.4932 effort=0.3 velocity=13.579; origin xyz=0 0 0.0290000000150089 rpy=0 0 0 -> xyz=0 0 0.0295 rpy=0 0 0
- joint finger4_tip_fixed: limit lower=0 upper=0 effort=100 velocity=10 -> (none); origin xyz=-0.00104042861977702 0 0.026700000917914 rpy=0 0 0 -> xyz=-0.0010528 0 0.0267 rpy=0 0 0
- joint finger5_joint1: axis 0 0.999999906157892 0.000433225353070638 -> 0 1 0; limit lower=-0.32695 upper=1.63595 effort=1 velocity=8.203047484 -> lower=-0.32695 upper=1.636 effort=1 velocity=8.203; origin xyz=-0.00226865106062467 -0.0340011106648613 0.0742813381426987 rpy=0.192050433506504 -0.0925172356498861 0.157672818297325 -> xyz=-0.0022687 -0.034001 0.074281 rpy=0.19248 -0.092517 0.15767
- joint finger5_joint2: limit lower=-0.495 upper=0.495 effort=0.2 velocity=8.115781022 -> lower=-0.495 upper=0.495 effort=0.2 velocity=8.1158; origin xyz=0.00220000070730803 0 0.00400000490038611 rpy=0.000433225364229257 0 0 -> xyz=0.0022 0 0.004 rpy=0 0 0
- joint finger5_joint3: axis -0 1 -0 -> 0 -1 0; limit lower=-0.4932 upper=1.6272 effort=0.3 velocity=12.86307659 -> lower=-1.6272 upper=0.4932 effort=0.3 velocity=12.863; origin xyz=-0.0046 1.5582E-05 0.036618 rpy=-0.00043323 0 -0.00026861 -> xyz=-0.00475 0 0.043618 rpy=0 0 -0.00026861
- joint finger5_joint4: axis -0 1 -0 -> 0 -1 0; limit lower=-0.4932 upper=1.6272 effort=0.3 velocity=13.57866158 -> lower=-1.6272 upper=0.4932 effort=0.3 velocity=13.579; origin xyz=0 0 0.029 rpy=0 0 0 -> xyz=0 0 0.0295 rpy=0 0 0
- joint finger5_tip_fixed: limit lower=0 upper=0 effort=100 velocity=10 -> (none); origin xyz=-0.00104042861181322 0 0.0267000011472218 rpy=0 0 0 -> xyz=-0.0010446 1.1308E-05 0.0267 rpy=0 0 0

Commit message: fix: Fix the incorrect direction of joint

File: urdf/left.urdf (robot description, URDF)
Before this commit: robot wujihand-left-v1.0.1, 26 links, 25 joints
Joints:
- joint finger1_joint1: axis 0 0 -1 -> 0 0 1; limit lower=-1.6508 upper=0.0448 effort=0.6 velocity=8.587 -> lower=-0.0448 upper=1.6508 effort=0.6 velocity=8.587
- joint finger2_joint2: axis 0 0 1 -> 0 0 -1
- joint finger2_joint3: axis 0 0 -1 -> 0 0 1; limit lower=-1.6272 upper=0.4932 effort=0.3 velocity=12.863 -> lower=-0.4932 upper=1.6272 effort=0.3 velocity=12.863
- joint finger2_joint4: axis 0 0 -1 -> 0 0 1; limit lower=-1.6272 upper=0.4932 effort=0.3 velocity=13.579 -> lower=-0.4932 upper=1.6272 effort=0.3 velocity=13.579
- joint finger3_joint1: axis -1 0 0 -> 1 0 0; limit lower=-1.63595 upper=0.32695 effort=1 velocity=8.203 -> lower=-0.32695 upper=1.63595 effort=1 velocity=8.203
- joint finger3_joint3: axis 0 0 -1 -> 0 0 1; limit lower=-1.6272 upper=0.4932 effort=0.3 velocity=12.863 -> lower=-0.4932 upper=1.6272 effort=0.3 velocity=12.863
- joint finger3_joint4: axis 0 0 -1 -> 0 0 1; limit lower=-1.6272 upper=0.4932 effort=0.3 velocity=13.579 -> lower=-0.4932 upper=1.6272 effort=0.3 velocity=13.579
- joint finger4_joint1: axis -1 0 0 -> 1 0 0; limit lower=-1.63595 upper=0.32695 effort=1 velocity=8.203 -> lower=-0.32695 upper=1.63595 effort=1 velocity=8.203
- joint finger4_joint3: axis 0 0 -1 -> 0 0 1; limit lower=-1.6272 upper=0.4932 effort=0.3 velocity=12.863 -> lower=-0.4932 upper=1.6272 effort=0.3 velocity=12.863
- joint finger4_joint4: axis 0 0 -1 -> 0 0 1; limit lower=-1.6272 upper=0.4932 effort=0.3 velocity=13.579 -> lower=-0.4932 upper=1.6272 effort=0.3 velocity=13.579
- joint finger5_joint3: axis 0 0 -1 -> 0 0 1; limit lower=-1.6272 upper=0.4932 effort=0.3 velocity=12.863 -> lower=-0.4932 upper=1.6272 effort=0.3 velocity=12.863

File: urdf/right.urdf (robot description, URDF)
Before this commit: robot wujihand-right-v1.0.1, 26 links, 25 joints
Joints:
- joint finger1_joint1: axis 0 -1 0 -> -0 1 -0; limit lower=-1.6508 upper=0.0448 effort=0.6 velocity=8.587 -> lower=-0.0448 upper=1.6508 effort=0.6 velocity=8.58701992
- joint finger1_joint2: axis 0 1 0 -> -0 -1 -0; limit lower=-0.9339 upper=0.1659 effort=0.6 velocity=11.1 -> lower=-0.1659 upper=0.9339 effort=0.6 velocity=11.10029404
- joint finger1_joint3: limit lower=-0.4932 upper=1.6272 effort=0.3 velocity=12.863 -> lower=-0.4932 upper=1.6272 effort=0.3 velocity=12.86307659
- joint finger1_joint4: limit lower=-0.4932 upper=1.6272 effort=0.3 velocity=13.579 -> lower=-0.4932 upper=1.6272 effort=0.3 velocity=13.57866158
- joint finger2_joint1: limit lower=-0.32695 upper=1.636 effort=1 velocity=8.203 -> lower=-0.32695 upper=1.63595 effort=1 velocity=8.203047484
- joint finger2_joint2: limit lower=-0.495 upper=0.495 effort=0.2 velocity=8.1158 -> lower=-0.495 upper=0.495 effort=0.2 velocity=8.115781022
- joint finger2_joint3: axis 0 -1 0 -> -0 1 -0; limit lower=-1.6272 upper=0.4932 effort=0.3 velocity=12.863 -> lower=-0.4932 upper=1.6272 effort=0.3 velocity=12.86307659
- joint finger2_joint4: axis 0 -1 0 -> -0 1 -0; limit lower=-1.6272 upper=0.4932 effort=0.3 velocity=13.579 -> lower=-0.4932 upper=1.6272 effort=0.3 velocity=13.57866158
- joint finger3_joint1: limit lower=-0.32695 upper=1.636 effort=1 velocity=8.203 -> lower=-0.32695 upper=1.63595 effort=1 velocity=8.203047484
- joint finger3_joint2: limit lower=-0.495 upper=0.495 effort=0.2 velocity=8.1158 -> lower=-0.495 upper=0.495 effort=0.2 velocity=8.115781022
- joint finger3_joint3: axis 0 -1 0 -> -0 1 -0; limit lower=-1.6272 upper=0.4932 effort=0.3 velocity=12.863 -> lower=-0.4932 upper=1.6272 effort=0.3 velocity=12.86307659
- joint finger3_joint4: axis 0 -1 0 -> -0 1 -0; limit lower=-1.6272 upper=0.4932 effort=0.3 velocity=13.579 -> lower=-0.4932 upper=1.6272 effort=0.3 velocity=13.57866158
- joint finger4_joint1: axis 0 -1 0 -> -0 1 -0; limit lower=-1.63595 upper=0.32695 effort=1 velocity=8.203 -> lower=-0.32695 upper=1.63595 effort=1 velocity=8.203047484
- joint finger4_joint2: limit lower=-0.495 upper=0.495 effort=0.2 velocity=8.1158 -> lower=-0.495 upper=0.495 effort=0.2 velocity=8.115781022
- joint finger4_joint3: axis 0 -1 0 -> -0 1 -0; limit lower=-1.6272 upper=0.4932 effort=0.3 velocity=12.863 -> lower=-0.4932 upper=1.6272 effort=0.3 velocity=12.86307659
- joint finger4_joint4: axis 0 -1 0 -> -0 1 -0; limit lower=-1.6272 upper=0.4932 effort=0.3 velocity=13.579 -> lower=-0.4932 upper=1.6272 effort=0.3 velocity=13.57866158
- joint finger5_joint1: limit lower=-0.32695 upper=1.636 effort=1 velocity=8.203 -> lower=-0.32695 upper=1.63595 effort=1 velocity=8.203047484
- joint finger5_joint2: limit lower=-0.495 upper=0.495 effort=0.2 velocity=8.1158 -> lower=-0.495 upper=0.495 effort=0.2 velocity=8.115781022
- joint finger5_joint3: axis 0 -1 0 -> -0 1 -0; limit lower=-1.6272 upper=0.4932 effort=0.3 velocity=12.863 -> lower=-0.4932 upper=1.6272 effort=0.3 velocity=12.86307659
- joint finger5_joint4: axis 0 -1 0 -> -0 1 -0; limit lower=-1.6272 upper=0.4932 effort=0.3 velocity=13.579 -> lower=-0.4932 upper=1.6272 effort=0.3 velocity=13.57866158
